File: pmi-hw-dan.kicad_pcb (KiCad board)
At the start: 2 copper layers, 56 x 20.3 mm, 26 parts, among them J1 Pmod-Interface-GPIO12, J2 Pmod-Interface-GPIO12, J3 Conn_01x06, Q1 IRLML6244, Q2 IRLML6244, Q3 IRLML6244, Q4 IRLML6244

Commit message: Bump to version 1.2
Parts:
- moved J3 2.29 mm to (109.5, 131.2)
Connections:
- net IO5 renamed /IO5
- net IO6 renamed /IO6
- net IO7 renamed /IO7
- net IO8 renamed /IO8
- net O5 renamed /O5
- net O6 renamed /O6
- net O7 renamed /O7
- net O8 renamed /O8
Routing:
- net /O8: track 10.5 -> 12.8 mm
- net /O7: track 4.86 -> 7.14 mm
- net /O6: track 9.80 -> 11.8 mm
- net +3.3V: track 45.1 -> 43.4 mm
- net /O5: track 14.1 -> 15.2 mm
- net GND: vias 15 -> 22
Other:
- board size 56 x 20.3 mm -> 55.9 x 20.3 mm
- board text added: "PMI-DAN V1.2"
- board text added: "PMI-DAN V1.2 2023"
- board text removed: "PMI-DAN V1.1"
- board text removed: "PMI-DAN V1.1 2022"
