File: pmi-hw-dan.kicad_sch (KiCad schematic)
At the start: 26 parts, among them J1 Pmod-Interface-GPIO12, J2 Pmod-Interface-GPIO12, J3 Conn_01x06, Q1 IRLML6244, Q2 IRLML6244, Q3 IRLML6244, Q4 IRLML6244

Commit message: Bump to version 1.2
Changed lines of the file:
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@@
   (title_block
     (title "PMI-DAN")
-    (date "2022-07-08")
-    (rev "V 1.0")
+    (date "2023-02-09")
+    (rev "V 1.2")
     (company "Paderborn University - Measurement Engineering Group")
   )
@@
     (effects (font (size 2.54 2.54)) (justify left bottom))
   )
-  (global_label "IO6" (shape bidirectional) (at 66.04 57.15 180) (fields_autoplaced)
-    (effects (font (size 1.27 1.27)) (justify right))
-    (property "Intersheet References" "${INTERSHEET_REFS}" (id 0) (at 60.4821 57.2294 0)
-      (effects (font (size 1.27 1.27)) (justify right) hide)
-    )
-  )
-  (global_label "IO5" (shape bidirectional) (at 49.53 54.61 0) (fields_autoplaced)
-    (effects (font (size 1.27 1.27)) (justify left))
-    (property "Intersheet References" "${INTERSHEET_REFS}" (id 0) (at 55.0879 54.5306 0)
-      (effects (font (size 1.27 1.27)) (justify left) hide)
-    )
-  )
-  (global_label "IO8" (shape bidirectional) (at 184.15 101.6 180) (fields_autoplaced)
-    (effects (font (size 1.27 1.27)) (justify right))
-    (property "Intersheet References" "${INTERSHEET_REFS}" (id 0) (at 178.5921 101.5206 0)
-      (effects (font (size 1.27 1.27)) (justify right) hide)
-    )
-  )
-  (global_label "IO6" (shape bidirectional) (at 49.53 57.15 0) (fields_autoplaced)
-    (effects (font (size 1.27 1.27)) (justify left))
-    (property "Intersheet References" "${INTERSHEET_REFS}" (id 0) (at 55.0879 57.0706 0)
-      (effects (font (size 1.27 1.27)) (justify left) hide)
-    )
-  )
-  (global_label "IO7" (shape bidirectional) (at 133.35 101.6 180) (fields_autoplaced)
-    (effects (font (size 1.27 1.27)) (justify right))
-    (property "Intersheet References" "${INTERSHEET_REFS}" (id 0) (at 127.7921 101.5206 0)
-      (effects (font (size 1.27 1.27)) (justify right) hide)
-    )
-  )
-  (global_label "O5" (shape input) (at 125.73 45.72 180) (fields_autoplaced)
-    (effects (font (size 1.27 1.27)) (justify right))
-    (property "Intersheet References" "${INTERSHEET_REFS}" (id 0) (at 120.7769 45.7994 0)
-      (effects (font (size 1.27 1.27)) (justify right) hide)
-    )
-  )
-  (global_label "IO8" (shape bidirectional) (at 66.04 62.23 180) (fields_autoplaced)
-    (effects (font (size 1.27 1.27)) (justify right))
-    (property "Intersheet References" "${INTERSHEET_REFS}" (id 0) (at 60.4821 62.3094 0)
-      (effects (font (size 1.27 1.27)) (justify right) hide)
-    )
-  )
-  (global_label "IO5" (shape bidirectional) (at 66.04 54.61 180) (fields_autoplaced)
-    (effects (font (size 1.27 1.27)) (justify right))
-    (property "Intersheet References" "${INTERSHEET_REFS}" (id 0) (at 60.4821 54.6894 0)
-      (effects (font (size 1.27 1.27)) (justify right) hide)
-    )
-  )
-  (global_label "O8" (shape input) (at 125.73 53.34 180) (fields_autoplaced)
-    (effects (font (size 1.27 1.27)) (justify right))
-    (property "Intersheet References" "${INTERSHEET_REFS}" (id 0) (at 120.7769 53.2606 0)
-      (effects (font (size 1.27 1.27)) (justify right) hide)
-    )
-  )
-  (global_label "IO5" (shape bidirectional) (at 33.02 101.6 180) (fields_autoplaced)
-    (effects (font (size 1.27 1.27)) (justify right))
-    (property "Intersheet References" "${INTERSHEET_REFS}" (id 0) (at 27.4621 101.6794 0)
-      (effects (font (size 1.27 1.27)) (justify right) hide)
-    )
-  )
-  (global_label "O6" (shape input) (at 125.73 48.26 180) (fields_autoplaced)
-    (effects (font (size 1.27 1.27)) (justify right))
-    (property "Intersheet References" "${INTERSHEET_REFS}" (id 0) (at 120.7769 48.1806 0)
-      (effects (font (size 1.27 1.27)) (justify right) hide)
-    )
-  )
-  (global_label "O5" (shape input) (at 57.15 92.71 0) (fields_autoplaced)
-    (effects (font (size 1.27 1.27)) (justify left))
-    (property "Intersheet References" "${INTERSHEET_REFS}" (id 0) (at 62.1031 92.6306 0)
-      (effects (font (size 1.27 1.27)) (justify left) hide)
-    )
-  )
-  (global_label "O6" (shape input) (at 106.68 92.71 0) (fields_autoplaced)
-    (effects (font (size 1.27 1.27)) (justify left))
-    (property "Intersheet References" "${INTERSHEET_REFS}" (id 0) (at 111.6331 92.6306 0)
-      (effects (font (size 1.27 1.27)) (justify left) hide)
-    )
-  )
-  (global_label "O8" (shape input) (at 208.28 92.71 0) (fields_autoplaced)
-    (effects (font (size 1.27 1.27)) (justify left))
-    (property "Intersheet References" "${INTERSHEET_REFS}" (id 0) (at 213.2331 92.6306 0)
-      (effects (font (size 1.27 1.27)) (justify left) hide)
-    )
-  )
-  (global_label "IO8" (shape bidirectional) (at 49.53 62.23 0) (fields_autoplaced)
-    (effects (font (size 1.27 1.27)) (justify left))
-    (property "Intersheet References" "${INTERSHEET_REFS}" (id 0) (at 55.0879 62.1506 0)
-      (effects (font (size 1.27 1.27)) (justify left) hide)
-    )
-  )
-  (global_label "O7" (shape input) (at 157.48 92.71 0) (fields_autoplaced)
-    (effects (font (size 1.27 1.27)) (justify left))
-    (property "Intersheet References" "${INTERSHEET_REFS}" (id 0) (at 162.4331 92.6306 0)
-      (effects (font (size 1.27 1.27)) (justify left) hide)
-    )
-  )
-  (global_label "IO7" (shape bidirectional) (at 49.53 59.69 0) (fields_autoplaced)
-    (effects (font (size 1.27 1.27)) (justify left))
-    (property "Intersheet References" "${INTERSHEET_REFS}" (id 0) (at 55.0879 59.6106 0)
-      (effects (font (size 1.27 1.27)) (justify left) hide)
-    )
-  )
-  (global_label "IO6" (shape bidirectional) (at 82.55 101.6 180) (fields_autoplaced)
-    (effects (font (size 1.27 1.27)) (justify right))
-    (property "Intersheet References" "${INTERSHEET_REFS}" (id 0) (at 76.9921 101.5206 0)
-      (effects (font (size 1.27 1.27)) (justify right) hide)
-    )
-  )
-  (global_label "IO7" (shape bidirectional) (at 66.04 59.69 180) (fields_autoplaced)
-    (effects (font (size 1.27 1.27)) (justify right))
-    (property "Intersheet References" "${INTERSHEET_REFS}" (id 0) (at 60.4821 59.7694 0)
-      (effects (font (size 1.27 1.27)) (justify right) hide)
-    )
-  )
-  (global_label "O7" (shape input) (at 125.73 50.8 180) (fields_autoplaced)
-    (effects (font (size 1.27 1.27)) (justify right))
-    (property "Intersheet References" "${INTERSHEET_REFS}" (id 0) (at 120.7769 50.7206 0)
-      (effects (font (size 1.27 1.27)) (justify right) hide)
-    )
+  (label "IO7" (at 133.35 101.6 180)
+    (effects (font (size 1.27 1.27)) (justify right bottom))
+  )
+  (label "IO6" (at 66.04 57.15 180)
+    (effects (font (size 1.27 1.27)) (justify right bottom))
+  )
+  (label "O6" (at 125.73 48.26 180)
+    (effects (font (size 1.27 1.27)) (justify right bottom))
+  )
+  (label "O5" (at 57.15 92.71 180)
+    (effects (font (size 1.27 1.27)) (justify right bottom))
+  )
+  (label "IO7" (at 66.04 59.69 180)
+    (effects (font (size 1.27 1.27)) (justify right bottom))
+  )
+  (label "O5" (at 125.73 45.72 180)
+    (effects (font (size 1.27 1.27)) (justify right bottom))
+  )
+  (label "O8" (at 125.73 53.34 180)
+    (effects (font (size 1.27 1.27)) (justify right bottom))
+  )
+  (label "IO8" (at 49.53 62.23 0)
+    (effects (font (size 1.27 1.27)) (justify left bottom))
+  )
+  (label "IO6" (at 49.53 57.15 0)
+    (effects (font (size 1.27 1.27)) (justify left bottom))
+  )
+  (label "IO5" (at 33.02 101.6 180)
+    (effects (font (size 1.27 1.27)) (justify right bottom))
+  )
+  (label "IO6" (at 82.55 101.6 180)
+    (effects (font (size 1.27 1.27)) (justify right bottom))
+  )
+  (label "IO5" (at 49.53 54.61 0)
+    (effects (font (size 1.27 1.27)) (justify left bottom))
+  )
+  (label "O7" (at 125.73 50.8 180)
+    (effects (font (size 1.27 1.27)) (justify right bottom))
+  )
+  (label "IO5" (at 66.04 54.61 180)
+    (effects (font (size 1.27 1.27)) (justify right bottom))
+  )
+  (label "O7" (at 157.48 92.71 180)
+    (effects (font (size 1.27 1.27)) (justify right bottom))
+  )
+  (label "O8" (at 208.28 92.71 180)
+    (effects (font (size 1.27 1.27)) (justify right bottom))
+  )
+  (label "IO7" (at 49.53 59.69 0)
+    (effects (font (size 1.27 1.27)) (justify left bottom))
+  )
+  (label "O6" (at 106.68 92.71 180)
+    (effects (font (size 1.27 1.27)) (justify right bottom))
+  )
+  (label "IO8" (at 184.15 101.6 180)
+    (effects (font (size 1.27 1.27)) (justify right bottom))
+  )
+  (label "IO8" (at 66.04 62.23 180)
+    (effects (font (size 1.27 1.27)) (justify right bottom))
   )
   (symbol (lib_id "Device:R") (at 187.96 106.68 0) (unit 1)
